File: DCDC.kicad_sch (KiCad schematic)
At the start: 21 parts, among them U50 TPS56A37RPAR, U51 AP7361-33E-13, U52 TLV741285PDBVR

Commit message: skdja7rkweg
Parts:
- removed C280, C281: 10uF, Capacitor_SMD:C_1206_3216Metric, symbol Capacitors:1206_uF10
- removed U51: AP7361-33E-13, DCDC:SOT-223_DIO, symbol DCDC:AP7361-33E-13
- removed U52: TLV741285PDBVR, DCDC:SOT23-5, symbol DCDC:TLV741285PDBVR
- added CB11: 100pF, Capacitor_SMD:C_0402_1005Metric, symbol Capacitors:0402_pF_100_50V
- L1: value WE-XHMI_7070 -> 74439387033
- RB1: renamed from R43; value 73.2K -> 73K2
- RB5: renamed from R47; value 73.2K -> 73K2
- renumbered R44 to RB2, R45 to RB3, R46 to RB4
Connections:
- net at RB4.1, RB5.2, U50.2 (FB): now also CB11.1
- net +5V renamed 5V
- net 5V: now also CB11.2
- no-connect marks 1 -> 0
Other:
- note removed: "Cin: 1uF Cout 1-100uF"
- note removed: "Cin: 1uF Cout 4.7uF+"
