File: Microwave_Beamer.kicad_pcb (KiCad board)
At the start: 4 copper layers, 179.5 x 180 mm, 448 parts, among them IC1 MAX2870ETJ+, U1 SKY13575-639LF, U10 SKY13575-639LF, U11 SKY13575-639LF, U12 SKY13575-639LF, U13 SE5023L-R, U14 SE5023L-R, U15 SE5023L-R, U16 SE5023L-R, U17 SE5023L-R, U18 SE5023L-R, U19 SE5023L-R, U2 SKY13575-639LF, U20 SE5023L-R, U21 SE5023L-R, U22 SE5023L-R, U23 SE5023L-R, U24 SE5023L-R, U25 SE5023L-R, U26 SE5023L-R, U27 SE5023L-R, U28 SE5023L-R, U29 SE5023L-R, U3 SKY13575-639LF, U30 SE5023L-R, U31 SE5023L-R, U32 SE5023L-R, U33 SE5023L-R, U34 SE5023L-R, U35 SE5023L-R, U36 SE5023L-R, U37 SE5023L-R, U38 SE5023L-R, U39 SE5023L-R, U4 SKY13575-639LF, U40 SE5023L-R, U41 SE5023L-R, U42 SE5023L-R, U43 SE5023L-R, U44 SE5023L-R, U45 SE5023L-R, U46 SE5023L-R, U47 SE5023L-R, U48 SE5023L-R, U49 SE5023L-R, U5 SKY13575-639LF, U50 TPS56A37RPAR, U51 AP7361-33E-13, U52 TLV741285PDBVR, U6 SKY13575-639LF, U7 SKY13575-639LF, U8 SKY13575-639LF, U9 SKY13575-639LF, Y1 ECS-3225MVQ-1000-CN-TR

Commit message: skdja7rkweg
Parts:
- removed C139, C151, C152, C153, C158, C160, C165, C166, C167, C172, C174, C179, C180, C181, C186, C188, C193, C194, C195, C200, C202, C207, C208, C209, C214, C216, C221, C222, C223, C228, C230, C235, C236, C237, C242, C244, C249, C250, C251, C256, C258: 1nF, Capacitor_SMD:C_0402_1005Metric
- removed C140, C147, C148, C149, C154, C155, C161, C162, C163, C168, C169, C175, C176, C177, C182, C183, C189, C190, C191, C196, C197, C203, C204, C205, C210, C211, C217, C218, C219, C224, C225, C231, C232, C233, C238, C239, C245, C246, C247, C252, C253, C259, C260, C261: 100pF, Capacitor_SMD:C_0402_1005Metric
- removed C156, C170, C184, C198, C212, C226, C240, C254, C262, C263, C264, C265, C266, C267, C268, C269, C270, C271, C272, C273, C274, C275, C276, C277, C278, C279: 100pFX, Capacitor_SMD:C_0402_1005Metric
- removed CB1, CB10, CB2, CB3, CB7, CB8, CB9: 10uF, Capacitor_SMD:C_1206_3216Metric
- removed CB4, CB5, CB6: 100nF, Capacitor_SMD:C_0603_1608Metric
- removed L1: WE-XHMI_7070, Inductors:WE-XHMI_7070
- removed U51: AP7361-33E-13, DCDC:SOT-223_DIO
- added C282: 100nF, Capacitor_SMD:C_0603_1608Metric, B.Cu at (170.8, 119.1)
- added C283: 1uF, Capacitor_SMD:C_0603_1608Metric, B.Cu at (-63.0, 21.5)
- added C284: 1uF, Capacitor_SMD:C_0603_1608Metric, B.Cu at (-57.0, 21.5)
- added C285: 10nF, Capacitor_SMD:C_0402_1005Metric, B.Cu at (35.2, 31.7)
- added C286: 10nF, Capacitor_SMD:C_0402_1005Metric, B.Cu at (87.2, 31.7)
- added C287: 10nF, Capacitor_SMD:C_0402_1005Metric, B.Cu at (139.2, 31.7)
- added C288: 10nF, Capacitor_SMD:C_0402_1005Metric, B.Cu at (35.2, 58.7)
- added C289: 10nF, Capacitor_SMD:C_0402_1005Metric, B.Cu at (87.2, 58.7)
- added C290: 10nF, Capacitor_SMD:C_0402_1005Metric, B.Cu at (139.2, 58.7)
- added C291: 10nF, Capacitor_SMD:C_0402_1005Metric, B.Cu at (35.2, 85.7)
- added C292: 10nF, Capacitor_SMD:C_0402_1005Metric, B.Cu at (87.2, 85.7)
- added C293: 10nF, Capacitor_SMD:C_0402_1005Metric, B.Cu at (139.2, 85.7)
- added C294: 10nF, Capacitor_SMD:C_0402_1005Metric, B.Cu at (35.2, 112.7)
- added C295: 10nF, Capacitor_SMD:C_0402_1005Metric, B.Cu at (87.2, 112.7)
- added C296: 10nF, Capacitor_SMD:C_0402_1005Metric, B.Cu at (139.2, 112.7)
- added C297: 10nF, Capacitor_SMD:C_0402_1005Metric, B.Cu at (35.2, 139.7)
- added C298: 10nF, Capacitor_SMD:C_0402_1005Metric, B.Cu at (87.2, 139.7)
- added C299: 10nF, Capacitor_SMD:C_0402_1005Metric, B.Cu at (139.2, 139.7)
- added C300: 10nF, Capacitor_SMD:C_0402_1005Metric, B.Cu at (35.2, 166.7)
- added C301: 10nF, Capacitor_SMD:C_0402_1005Metric, B.Cu at (87.2, 166.7)
- added C302: 10nF, Capacitor_SMD:C_0402_1005Metric, B.Cu at (139.2, 166.7)
- added C303: 10nF, Capacitor_SMD:C_0402_1005Metric, B.Cu at (180.6, 38.2)
- added C304: 10nF, Capacitor_SMD:C_0402_1005Metric, B.Cu at (40.9, 31.3)
- added C305: 10nF, Capacitor_SMD:C_0402_1005Metric, B.Cu at (92.8, 31.3)
- added C306: 10nF, Capacitor_SMD:C_0402_1005Metric, B.Cu at (144.8, 31.3)
- added C307: 10nF, Capacitor_SMD:C_0402_1005Metric, B.Cu at (40.9, 58.3)
- added C308: 10nF, Capacitor_SMD:C_0402_1005Metric, B.Cu at (144.8, 58.3)
- added C309: 10nF, Capacitor_SMD:C_0402_1005Metric, B.Cu at (92.8, 58.3)
- added C310: 10nF, Capacitor_SMD:C_0402_1005Metric, B.Cu at (40.9, 85.3)
- added C311: 10nF, Capacitor_SMD:C_0402_1005Metric, B.Cu at (144.8, 85.3)
- added C312: 10nF, Capacitor_SMD:C_0402_1005Metric, B.Cu at (92.8, 85.3)
- added C313: 10nF, Capacitor_SMD:C_0402_1005Metric, B.Cu at (40.9, 112.3)
- added C314: 10nF, Capacitor_SMD:C_0402_1005Metric, B.Cu at (144.8, 112.3)
- added C315: 10nF, Capacitor_SMD:C_0402_1005Metric, B.Cu at (92.8, 112.3)
- added C316: 10nF, Capacitor_SMD:C_0402_1005Metric, B.Cu at (40.9, 139.3)
- added C317: 10nF, Capacitor_SMD:C_0402_1005Metric, B.Cu at (144.8, 139.3)
- added C318: 10nF, Capacitor_SMD:C_0402_1005Metric, B.Cu at (92.8, 139.3)
- added C319: 10nF, Capacitor_SMD:C_0402_1005Metric, B.Cu at (40.9, 166.3)
- added C320: 10nF, Capacitor_SMD:C_0402_1005Metric, B.Cu at (144.8, 166.3)
- added C321: 10nF, Capacitor_SMD:C_0402_1005Metric, B.Cu at (92.8, 166.3)
- added C322: 100nF, Capacitor_SMD:C_0603_1608Metric, B.Cu at (176.0, 128.5)
- added C323: 100nF, Capacitor_SMD:C_0402_1005Metric, B.Cu at (180.0, 115.5)
- added C324: 100nF, Capacitor_SMD:C_0402_1005Metric, B.Cu at (181.5, 117.0)
- added C325: 100nF, Capacitor_SMD:C_0402_1005Metric, B.Cu at (173.5, 118.7)
- added C326: 100nF, Capacitor_SMD:C_0402_1005Metric, B.Cu at (178.6, 124.2)
- added C327: 100nF, Capacitor_SMD:C_0402_1005Metric, B.Cu at (173.5, 123.4)
- added C328: 100nF, Capacitor_SMD:C_0402_1005Metric, B.Cu at (174.5, 115.5)
- added CB13: 10uF, Capacitor_SMD:C_1206_3216Metric, B.Cu at (262.5, 118.7)
- added L4: IHLP6767GZERR47M11, Inductors:IND_IHLP-6767GZ_VIS, B.Cu at (178.5, 77.3)
- added PS1: R-78K5.0-1.0, DCDC:DCDC_R-78K3.3-0.5, F.Cu at (237.9, 140.1)
- added R48: 10K, Resistor_SMD:R_0603_1608Metric, B.Cu at (186.7, 121.5)
- added R49: 24.9k, Resistor_SMD:R_0603_1608Metric, B.Cu at (183.5, 58.8)
- added R50: x, Resistor_SMD:R_0603_1608Metric, B.Cu at (182.0, 58.8)
- added R51: x, Resistor_SMD:R_0603_1608Metric, B.Cu at (177.5, 58.8)
- added R52: 10K, Resistor_SMD:R_0603_1608Metric, B.Cu at (185.2, 121.5)
- added R53: 10K, Resistor_SMD:R_0603_1608Metric, B.Cu at (182.7, 126.5)
- added R54: 10K, Resistor_SMD:R_0603_1608Metric, B.Cu at (182.7, 125.0)
- added R55: 10K, Resistor_SMD:R_0603_1608Metric, B.Cu at (185.7, 125.0)
- added U55: TPS548D26RXXR, DCDC:WQFN_C26RXXR_TEX, B.Cu at (181.2, 63.9)
- C100, C58, C72, C86: value 100pFX -> 1uF; footprint Capacitor_SMD:C_0402_1005Metric -> Capacitor_SMD:C_0603_1608Metric
- C102, C104, C109, C116, C123, C124, C137, C138, C53, C54, C55, C60, C62, C67, C68, C69, C74, C76, C83, C88, C90, C97: value 1nF -> 1uF; footprint Capacitor_SMD:C_0402_1005Metric -> Capacitor_SMD:C_0603_1608Metric
- C105, C112, C120, C134, C135, C51, C56, C57, C63, C64, C65, C77, C78, C79, C91, C92, C93: value 100pF -> 1uF; footprint Capacitor_SMD:C_0402_1005Metric -> Capacitor_SMD:C_0603_1608Metric
- C106, C113, C15, C22, C36, C70, C84, C98: value 100pF -> 1nF
- C107, C119, C121, C14, C21, C28, C29, C30, C35, C42, C43, C44, C49, C50, C7, C71, C8, C85, C9, C99: value 100pF -> 100nF; footprint Capacitor_SMD:C_0402_1005Metric -> Capacitor_SMD:C_0603_1608Metric
- C111, C12, C125, C19, C25, C27, C33, C39, C4, C41, C46, C48, C6, C82, C96: value 1nF -> 100nF; footprint Capacitor_SMD:C_0402_1005Metric -> Capacitor_SMD:C_0603_1608Metric
- C114, C16, C23, C37: value 100pFX -> 100nF; footprint Capacitor_SMD:C_0402_1005Metric -> Capacitor_SMD:C_0603_1608Metric
- C126, C127, C133: value 100pF -> 10uF; footprint Capacitor_SMD:C_0402_1005Metric -> Capacitor_SMD:C_1206_3216Metric
- C128: value 100pFX -> 10uF; footprint Capacitor_SMD:C_0402_1005Metric -> Capacitor_SMD:C_1206_3216Metric
- C130, C132: value 1nF -> 10uF; footprint Capacitor_SMD:C_0402_1005Metric -> Capacitor_SMD:C_1206_3216Metric
- C141: value 100pF -> 47uF; footprint Capacitor_SMD:C_0402_1005Metric -> Capacitor_SMD:C_1206_3216Metric
- C142: value 100pFX -> 47uF; footprint Capacitor_SMD:C_0402_1005Metric -> Capacitor_SMD:C_1206_3216Metric
- C144, C146: value 1nF -> 47uF; footprint Capacitor_SMD:C_0402_1005Metric -> Capacitor_SMD:C_1206_3216Metric
- C280: value 10uF -> 1nF; footprint Capacitor_SMD:C_1206_3216Metric -> Capacitor_SMD:C_0402_1005Metric; moved to B.Cu
- C281: value 10uF -> 100nF; footprint Capacitor_SMD:C_1206_3216Metric -> Capacitor_SMD:C_0603_1608Metric; moved to B.Cu
- R43: value 73.2K -> 33; footprint Resistor_SMD:R_0603_1608Metric -> Resistor_SMD:R_0402_1005Metric; moved to B.Cu
- R44: value 52.3k -> 250; moved to B.Cu
- R45: value 10K -> 100; footprint Resistor_SMD:R_0603_1608Metric -> Resistor_SMD:R_0402_1005Metric; moved to B.Cu
- R46, R47: moved to B.Cu
- U50: value TPS56A37RPAR -> LDL1117S33R; footprint DCDC:DCDC_RPA0010A-MFG -> DCDC:SOT-223_DIO
- U52: value TLV741285PDBVR -> MIC5219-2.85YM5-TR
- moved W2 374.4 mm to (260.5, 55.0)
- moved R2 374.4 mm to (255.3, 55.0)
- moved R4 372.5 mm to (229.9, 60.0)
- moved R5 372.5 mm to (253.3, 60.0)
- moved W4 372.5 mm to (235.1, 60.0)
- moved W5 372.5 mm to (248.1, 60.0)
- moved W1 370.0 mm to (243.5, 50.0), turned to 180 degrees
- moved R1 359.5 mm to (238.3, 50.0), turned to -90 degrees
- moved C130 155.6 mm to (175.0, 60.3), turned to 90 degrees
- moved C50 153.4 mm to (180.5, 40.7)
- moved C133 152.2 mm to (171.0, 60.3), turned to 90 degrees
- moved C49 151.1 mm to (139.1, 169.2), turned to 180 degrees
- moved C42 146.9 mm to (35.1, 142.2)
- moved C135 146.7 mm to (182.2, 121.5), turned to 180 degrees
- moved C132 146.7 mm to (173.0, 60.3), turned to 90 degrees
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Connections:
- C102 pad 1: +5V -> /STEM/FAN_F/POWER AMP3/VCC
- C103 pad 1: +5V -> /STEM/FAN_C/POWER AMP3/VCC
- C121 pad 1: +5V -> Net-(U55-BOOT)
- C121 pad 2: GND -> Net-(U55-PHASE)
- C123 pad 1: +5V -> 5V_LP
- C124 pad 1: +5V -> 5V_LP
- C125 pad 1: +5V -> +12V
- C126 pad 1: +5V -> +12V
- C127 pad 1: +5V -> +12V
- C128 pad 1: +5V -> +12V
- C130 pad 1: +5V -> +12V
- C132 pad 1: +5V -> +12V
- C133 pad 1: +5V -> +12V
- C135 pad 1: +5V -> GND
- C135 pad 2: GND -> Net-(IC1-BIAS_FILT)
- C137 pad 1: +5V -> GND
- C137 pad 2: GND -> Net-(IC1-NOISE_FILT)
- C138 pad 1: +5V -> GND
- C138 pad 2: GND -> Net-(IC1-REG)
- C145 pad 1: +5V -> /STEM/FAN_D/POWER AMP3/VCC
- C187 pad 1: +5V -> /STEM/FAN_E/POWER AMP3/VCC
- C229 pad 1: +5V -> /STEM/FAN_F/POWER AMP3/VCC
- C26 pad 1: +5V -> /STEM/FAN_A/POWER AMP3/VCC
- C28 pad 1: +5V -> /STEM/FAN_C/POWER AMP3/VCC
- C280 pad 1: +5V -> Net-(IC1-TUNE)
- C281 pad 1: +3.3V -> Net-(IC1-CP_OUT)
- C281 pad 2: GND -> Net-(C281-Pad2)
- C39 pad 1: +5V -> /STEM/FAN_D/POWER AMP3/VCC
- C43 pad 1: +5V -> /STEM/FAN_E/POWER AMP3/VCC
- C48 pad 1: +5V -> /STEM/FAN_F/POWER AMP3/VCC
- C6 pad 1: +5V -> /STEM/FAN_A/POWER AMP3/VCC
- C60 pad 1: +5V -> /STEM/FAN_A/POWER AMP3/VCC
- C61 pad 1: +5V -> /STEM/FAN_B/POWER AMP3/VCC
- C64 pad 1: +5V -> /STEM/FAN_B/POWER AMP3/VCC
- C76 pad 1: +5V -> /STEM/FAN_C/POWER AMP3/VCC
- C79 pad 1: +5V -> /STEM/FAN_D/POWER AMP3/VCC
- C9 pad 1: +5V -> /STEM/FAN_B/POWER AMP3/VCC
- C91 pad 1: +5V -> /STEM/FAN_E/POWER AMP3/VCC
- IC1 pad 19: unconnected-(IC1-NOISE_FILT-Pad19) -> Net-(IC1-NOISE_FILT)
- IC1 pad 20: unconnected-(IC1-TUNE-Pad20) -> Net-(IC1-TUNE)
- IC1 pad 22: unconnected-(IC1-RSET-Pad22) -> Net-(IC1-RSET)
- IC1 pad 23: unconnected-(IC1-BIAS_FILT-Pad23) -> Net-(IC1-BIAS_FILT)
- IC1 pad 24: unconnected-(IC1-REG-Pad24) -> Net-(IC1-REG)
- IC1 pad 25: unconnected-(IC1-LD-Pad25) -> Net-(IC1-LD)
- IC1 pad 26: unconnected-(IC1-RFOUT_EN-Pad26) -> Net-(IC1-RFOUT_EN)
- IC1 pad 4: unconnected-(IC1-CE-Pad4) -> +3.3V
- IC1 pad 5: unconnected-(IC1-SW-Pad5) -> Net-(IC1-SW)
- IC1 pad 7: unconnected-(IC1-CP_OUT-Pad7) -> Net-(IC1-CP_OUT)
- R43 pad 1: /DCDC/24V -> Net-(C281-Pad2)
- R43 pad 2: Net-(U50-EN) -> Net-(IC1-SW)
- R44 pad 1: Net-(U50-MODE) -> Net-(IC1-CP_OUT)
- R44 pad 2: GND -> Net-(IC1-TUNE)
- R45 pad 1: Net-(U50-EN) -> Net-(IC1-SW)
- R46 pad 1: Net-(U50-FB) -> Net-(U55-FB)
- R47 pad 1: +5V -> Net-(U55-FB)
- R47 pad 2: Net-(U50-FB) -> +5V
- U13 pad 10: unconnected-(U13-DETECT-Pad10) -> /STEM/FAN_A/POWER AMP1/power detect
- U16 pad 10: unconnected-(U16-DETECT-Pad10) -> /STEM/FAN_A/POWER AMP3/power detect
- U16 pad 18: +5V -> /STEM/FAN_A/POWER AMP3/VCC
- U16 pad 19: +5V -> /STEM/FAN_A/POWER AMP3/VCC
- U16 pad 20: +5V -> /STEM/FAN_A/POWER AMP3/VCC
- U16 pad 8: +5V -> /STEM/FAN_A/POWER AMP3/VCC
- U16 pad 9: +5V -> /STEM/FAN_A/POWER AMP3/VCC
- U18 pad 10: unconnected-(U18-DETECT-Pad10) -> /STEM/FAN_A/POWER AMP5/power detect
- U19 pad 10: unconnected-(U19-DETECT-Pad10) -> /STEM/FAN_B/POWER AMP1/power detect
- U21 pad 10: unconnected-(U21-DETECT-Pad10) -> /STEM/FAN_B/POWER AMP3/power detect
- U21 pad 18: +5V -> /STEM/FAN_B/POWER AMP3/VCC
- U21 pad 19: +5V -> /STEM/FAN_B/POWER AMP3/VCC
- U21 pad 20: +5V -> /STEM/FAN_B/POWER AMP3/VCC
- U21 pad 8: +5V -> /STEM/FAN_B/POWER AMP3/VCC
- U21 pad 9: +5V -> /STEM/FAN_B/POWER AMP3/VCC
- U23 pad 10: unconnected-(U23-DETECT-Pad10) -> /STEM/FAN_B/POWER AMP5/power detect
- U25 pad 10: unconnected-(U25-DETECT-Pad10) -> /STEM/FAN_C/POWER AMP1/power detect
- U27 pad 10: unconnected-(U27-DETECT-Pad10) -> /STEM/FAN_C/POWER AMP3/power detect
- U27 pad 18: +5V -> /STEM/FAN_C/POWER AMP3/VCC
- U27 pad 19: +5V -> /STEM/FAN_C/POWER AMP3/VCC
- U27 pad 20: +5V -> /STEM/FAN_C/POWER AMP3/VCC
- U27 pad 8: +5V -> /STEM/FAN_C/POWER AMP3/VCC
- U27 pad 9: +5V -> /STEM/FAN_C/POWER AMP3/VCC
- U29 pad 10: unconnected-(U29-DETECT-Pad10) -> /STEM/FAN_C/POWER AMP5/power detect
- U31 pad 10: unconnected-(U31-DETECT-Pad10) -> /STEM/FAN_D/POWER AMP1/power detect
- U33 pad 10: unconnected-(U33-DETECT-Pad10) -> /STEM/FAN_D/POWER AMP3/power detect
- U33 pad 18: +5V -> /STEM/FAN_D/POWER AMP3/VCC
- U33 pad 19: +5V -> /STEM/FAN_D/POWER AMP3/VCC
- U33 pad 20: +5V -> /STEM/FAN_D/POWER AMP3/VCC
- U33 pad 8: +5V -> /STEM/FAN_D/POWER AMP3/VCC
- U33 pad 9: +5V -> /STEM/FAN_D/POWER AMP3/VCC
- U35 pad 10: unconnected-(U35-DETECT-Pad10) -> /STEM/FAN_D/POWER AMP5/power detect
- U37 pad 10: unconnected-(U37-DETECT-Pad10) -> /STEM/FAN_E/POWER AMP1/power detect
- U39 pad 10: unconnected-(U39-DETECT-Pad10) -> /STEM/FAN_E/POWER AMP3/power detect
- U39 pad 18: +5V -> /STEM/FAN_E/POWER AMP3/VCC
- U39 pad 19: +5V -> /STEM/FAN_E/POWER AMP3/VCC
- U39 pad 20: +5V -> /STEM/FAN_E/POWER AMP3/VCC
- U39 pad 8: +5V -> /STEM/FAN_E/POWER AMP3/VCC
- U39 pad 9: +5V -> /STEM/FAN_E/POWER AMP3/VCC
- U41 pad 10: unconnected-(U41-DETECT-Pad10) -> /STEM/FAN_E/POWER AMP5/power detect
- U43 pad 10: unconnected-(U43-DETECT-Pad10) -> /STEM/FAN_F/POWER AMP1/power detect
- U45 pad 10: unconnected-(U45-DETECT-Pad10) -> /STEM/FAN_F/POWER AMP3/power detect
- U45 pad 18: +5V -> /STEM/FAN_F/POWER AMP3/VCC
- U45 pad 19: +5V -> /STEM/FAN_F/POWER AMP3/VCC
- U45 pad 20: +5V -> /STEM/FAN_F/POWER AMP3/VCC
- U45 pad 8: +5V -> /STEM/FAN_F/POWER AMP3/VCC
- U45 pad 9: +5V -> /STEM/FAN_F/POWER AMP3/VCC
- U47 pad 10: unconnected-(U47-DETECT-Pad10) -> /STEM/FAN_F/POWER AMP5/power detect
- U49 pad 10: unconnected-(U49-DETECT-Pad10) -> /POWER AMP6/power detect
- U50 pad 1: Net-(U50-EN) -> GND
- U50 pad 2: Net-(U50-FB) -> +3.3V
- U50 pad 3: GND -> 5V_LP
- U50 pad 4: unconnected-(U50-PG-Pad4) -> +3.3V
- U52 pad 3: +3.3V -> /POWER/AMP_enable
- Y1 pad 1: unconnected-(Y1-~{EN}-Pad1) -> GND
Routing:
- net +5V: track 618.5 -> 688.7 mm, vias 111 -> 62
- net /STEM/FAN_A/POWER AMP3/VCC: track 0.00 -> 22.0 mm, vias 0 -> 2
- net /STEM/FAN_F/POWER AMP3/VCC: track 0.00 -> 22.0 mm, vias 0 -> 2
- net /STEM/FAN_E/POWER AMP3/VCC: track 0.00 -> 22.0 mm, vias 0 -> 2
- net /STEM/FAN_D/POWER AMP3/VCC: track 0.00 -> 22.0 mm, vias 0 -> 2
- net /STEM/FAN_C/POWER AMP3/VCC: track 0.00 -> 22.0 mm, vias 0 -> 2
- net /STEM/FAN_B/POWER AMP3/VCC: track 0.00 -> 22.0 mm, vias 0 -> 2
- net 2.85VREF: track 304.4 -> 324.4 mm
- net GND: track 176.4 -> 194.3 mm, vias 861 -> 860
- net /POWER AMP6/RF_OUT: track 44.0 -> 49.0 mm
- net Net-(U55-FB): track 0.00 -> 4.26 mm
- net 5V_LP: track 0.00 -> 3.25 mm
- net Net-(U55-SS): track 0.00 -> 2.57 mm
- net Net-(U55-BOOT): track 0.00 -> 2.56 mm
- net Net-(U55-MODE): track 0.00 -> 2.17 mm
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
Commit message: moving along
Parts:
- removed C281, C282: 100nF, Capacitor_SMD:C_0603_1608Metric
- added ?: , , F.Cu at (205.0, 129.0)
- added ?: , , F.Cu at (205.0, 145.0)
- added ?: , , F.Cu at (180.0, 105.0)
- added ?: , , F.Cu at (200.0, 75.0)
- added ?: , , F.Cu at (200.0, 105.0)
- added ?: , , F.Cu at (205.0, 137.0)
- added ?: , , F.Cu at (180.0, 75.0)
- added C329: 100nF, Capacitor_SMD:C_0402_1005Metric, B.Cu at (173.2, 41.3)
- added C330: 100nF, Capacitor_SMD:C_0402_1005Metric, B.Cu at (172.1, 43.3)
- added D1: LTST-C230KGKT, LED_SMD:LED_1206_3216Metric, B.Cu at (163.1, 144.5)
- added D2: LTST-C230KGKT, LED_SMD:LED_1206_3216Metric, B.Cu at (162.5, 148.0)
- added D3: LTST-C230KGKT, LED_SMD:LED_1206_3216Metric, B.Cu at (163.8, 153.0)
- added D4: LTST-C230KGKT, LED_SMD:LED_1206_3216Metric, B.Cu at (165.5, 140.9)
- added D5: LTST-C230KGKT, LED_SMD:LED_1206_3216Metric, F.Cu at (234.9, 96.5)
- added D6: LTST-C230KGKT, LED_SMD:LED_1206_3216Metric, F.Cu at (235.0, 83.5)
- added G***: LOGO, Graphics:Radiation_danger, F.Cu at (225.9, 89.9)
- added R56: 250, Resistor_SMD:R_0603_1608Metric, B.Cu at (164.0, 160.9)
- added R57: 250, Resistor_SMD:R_0603_1608Metric, B.Cu at (162.0, 160.9)
- added R58: 250, Resistor_SMD:R_0603_1608Metric, B.Cu at (160.0, 160.9)
- added R59: 250, Resistor_SMD:R_0603_1608Metric, B.Cu at (166.0, 160.9)
- added R60: 100, Resistor_SMD:R_0402_1005Metric, B.Cu at (245.9, 135.2)
- added R61: 100, Resistor_SMD:R_0402_1005Metric, B.Cu at (245.9, 137.2)
- added U51: SN74LVC1G14DCKR, Logic:SOT65P210X110-5N, B.Cu at (172.2, 163.5)
- added U53: SN74LVC1G14DCKR, Logic:SOT65P210X110-5N, B.Cu at (172.2, 168.0)
- added U54: 74HC138D, Logic:SOT109-1_NXP, B.Cu at (164.0, 166.9)
- added U56: PI_PICO, Logic:PI_PICO_SMD, B.Cu at (182.4, 17.3)
- added U57: SN74LVC1G14DCKR, Logic:SOT65P210X110-5N, B.Cu at (243.5, 92.2)
- PS1, U50, U52: moved to B.Cu
- moved W3 268.2 mm to (160.0, 109.5), turned to -90 degrees
- moved R3 263.6 mm to (160.0, 114.7), turned to 0 degrees
- moved C284 257.4 mm to (199.5, 42.5), turned to -90 degrees
- moved C283 254.5 mm to (190.7, 41.0), turned to 90 degrees
- moved W6 218.9 mm to (153.0, 122.5), turned to -90 degrees
- moved R6 214.8 mm to (153.0, 127.7), turned to 0 degrees
- moved PS1 113.3 mm to (185.7, 39.5), turned to -90 degrees
- moved R51 111.2 mm to (188.0, 169.5), turned to -90 degrees
- moved R47 111.0 mm to (186.5, 169.5), turned to -90 degrees
- moved R46 110.8 mm to (185.0, 169.5), turned to 90 degrees
- moved R49 110.7 mm to (182.0, 169.5), turned to -90 degrees
- moved R50 110.7 mm to (183.5, 169.5), turned to -90 degrees
- moved U50 110.3 mm to (197.0, 36.5), turned to -90 degrees
- moved C133 110.3 mm to (194.5, 168.0), turned to -90 degrees
- moved C132 109.5 mm to (192.5, 168.0), turned to -90 degrees
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Connections:
- net Net-(IC1-RFOUT_EN) renamed /RF_EN
- IC1 pad 1: unconnected-(IC1-CLK-Pad1) -> CLK
- IC1 pad 2: unconnected-(IC1-DATA-Pad2) -> /MOSI
- IC1 pad 3: unconnected-(IC1-LE-Pad3) -> /LE
- IC1 pad 4: +3.3V -> /Chip_EN
- RR1 pad 1: 3V3 -> +3.3V
- RR2 pad 1: 3V3 -> +3.3V
- U18 pad 10: /STEM/FAN_A/POWER AMP5/power detect -> Stage_2_power
- U23 pad 10: /STEM/FAN_B/POWER AMP5/power detect -> Stage_2_power
- U29 pad 10: /STEM/FAN_C/POWER AMP5/power detect -> Stage_2_power
- U35 pad 10: /STEM/FAN_D/POWER AMP5/power detect -> Stage_2_power
- U41 pad 10: /STEM/FAN_E/POWER AMP5/power detect -> Stage_2_power
- U47 pad 10: /STEM/FAN_F/POWER AMP5/power detect -> Stage_2_power
- U49 pad 10: /POWER AMP6/power detect -> Stage_1_power
- U52 pad 3: /POWER/AMP_enable -> /AMP_enable
Routing:
- net (no net): track 84.1 -> 24.1 mm, vias 22 -> 20
- net Net-(U6-RFC): track 5.62 -> 55.6 mm
- net Net-(U4-RFC): track 5.62 -> 52.2 mm
- net /POWER AMP6/RF_OUT: track 49.0 -> 3.97 mm, vias 1 -> 0
- net /STEM/FAN_A/Antenna_1: track 21.2 -> 56.2 mm
- net Net-(U3-RFC): track 5.62 -> 38.2 mm
- net Net-(U5-RFC): track 5.62 -> 37.4 mm
- net Net-(W1-Out2): track 5.62 -> 36.3 mm
- net Net-(W2-Out2): track 5.62 -> 26.2 mm
- net Net-(W2-Out1): track 5.62 -> 24.5 mm
- net /STEM/FAN_B/Antenna_2: track 32.8 -> 14.5 mm
- net /STEM/FAN_F/Antenna_2: track 32.8 -> 14.5 mm
- net /STEM/FAN_E/Antenna_6: track 32.8 -> 14.5 mm
- net /STEM/FAN_E/Antenna_2: track 32.8 -> 14.5 mm
- net /STEM/FAN_D/Antenna_2: track 32.8 -> 14.5 mm
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Other:
- board size 179.5 x 180 mm -> 200 x 170 mm
- board text added: "-30^{o}"
- board text added: "0^{o}"
- board text added: "20^{o}"
- board text added: "45^{o}"
- board text added: "BEAM ANGLE"
- board text added: "Danger Radiation"
