File: dcdc30A.kicad_sch (KiCad schematic)
At the start: 22 parts, among them U55 TPS548D26RXXR

Commit message: moving along
Changed lines of the file:
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@@
 	)
 	(junction
+		(at 142.24 96.52)
+		(diameter 0)
+		(color 0 0 0 0)
+	)
+	(junction
 		(at 121.92 86.36)
 		(diameter 0)
@@
 	)
 	(junction
-		(at 142.24 96.52)
-		(diameter 0)
-		(color 0 0 0 0)
-	)
-	(junction
 		(at 63.5 104.14)
 		(diameter 0)
@@
 	(wire
 		(pts
-			(xy 149.86 91.44) (xy 142.24 91.44)
-		)
-		(stroke
-			(width 0)
-			(type default)
-		)
-	)
-	(wire
-		(pts
 			(xy 172.72 88.9) (xy 177.8 88.9)
 		)
@@
 	(wire
 		(pts
-			(xy 149.86 88.9) (xy 149.86 91.44)
+			(xy 149.86 88.9) (xy 149.86 96.52)
 		)
 		(stroke
@@
 	(wire
 		(pts
-			(xy 142.24 91.44) (xy 142.24 96.52)
-		)
-		(stroke
-			(width 0)
-			(type default)
-		)
-	)
-	(wire
-		(pts
 			(xy 149.86 88.9) (xy 147.32 88.9)
 		)
@@
 	(wire
 		(pts
+			(xy 149.86 96.52) (xy 142.24 96.52)
+		)
+		(stroke
+			(width 0)
+			(type default)
+		)
+	)
+	(wire
+		(pts
 			(xy 48.26 83.82) (xy 53.34 83.82)
 		)
@@
 		)
 		(property "Value" "73.2K"
-			(at 142.24 101.6 90)
+			(at 140.97 101.6 90)
 			(show_name no)
 			(do_not_autoplace yes)
