File: pico.kicad_sch (KiCad schematic)
At the start: 0 parts

Commit message: moving along
Parts:
- added D1, D2, D3, D4: LTST-C230KGKT, LED_SMD:LED_1206_3216Metric, symbol LED:IR26-21C_L110_TR8
- added R56, R57, R58, R59: 250, Resistor_SMD:R_0603_1608Metric, symbol Resistors:R
- added U51, U53: SN74LVC1G14DCKR, Logic:SOT65P210X110-5N, symbol Logic:SN74LVC1G14DCKR
- added U54: 74HC138D, Logic:SOT109-1_NXP, symbol Logic:74HC138D
Connections:
- new net: D4.1 (K), R59.1
- new net: D2.1 (K), R57.1
- new net: D1.1 (K), R56.1
- new net: D3.1 (K), R58.1
- new net +3.3V: U51.5 (VCC), U53.5 (VCC)
- new net 5V_LP: D1.2 (A), D2.2 (A), D3.2 (A), D4.2 (A), U54.16 (VCC)
- new net AMP_enable: U54.6 (E3)
- new net GND: U51.3 (GND), U53.3 (GND), U54.3 (A2), U54.4 (E*1), U54.5 (E*2), U54.8 (GND)
- new net PHASE_CTRL_1: U51.2 (A), U54.2 (A1)
- new net PHASE_CTRL_2: U53.2 (A), U54.1 (A0)
- new net led_n20: R56.2, U54.15 (Y*0)
- new net led_n45: R59.2, U54.12 (Y*3)
- new net led_p30: R58.2, U54.13 (Y*2)
- new net led_zero: R57.2, U54.14 (Y*1)
- new net ~{PHASE_CTRL_1}: U51.4 (Y)
- new net ~{PHASE_CTRL_2}: U53.4 (Y)
- no-connect marks 0 -> 4
