File: FANFAN.kicad_sch (KiCad schematic)
At the start: 13 parts

Commit message: skdja7rkweg
Parts:
- W10, W11, W12, W7, W8, W9: value ~ -> (none)

Commit message: 6 layers now
Parts:
- R10, R11, R12, R7, R8, R9, RL2: price (none) -> .04
Changed lines of the file:
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@@
+			)
+		)
+		(property "price" ".04"
+			(at 144.78 73.66 0)
+			(hide yes)
+			(show_name no)
+			(do_not_autoplace no)
+			(effects
+				(font
+					(size 1.27 1.27)
+				)
 			)
 		)
@@
 			)
 		)
+		(property "price" ".04"
+			(at 119.38 109.22 0)
+			(hide yes)
+			(show_name no)
+			(do_not_autoplace no)
+			(effects
+				(font
+					(size 1.27 1.27)
+				)
+			)
+		)
 		(pin "1"
 		)
@@
 			)
 		)
+		(property "price" ".04"
+			(at 144.78 53.34 0)
+			(hide yes)
+			(show_name no)
+			(do_not_autoplace no)
+			(effects
+				(font
+					(size 1.27 1.27)
+				)
+			)
+		)
 		(pin "1"
 		)
@@
 			)
 		)
+		(property "price" ".04"
+			(at 119.38 60.96 0)
+			(hide yes)
+			(show_name no)
+			(do_not_autoplace no)
+			(effects
+				(font
+					(size 1.27 1.27)
+				)
+			)
+		)
 		(pin "1"
 		)
@@
 			)
 		)
+		(property "price" ".04"
+			(at 144.78 101.6 0)
+			(hide yes)
+			(show_name no)
+			(do_not_autoplace no)
+			(effects
+				(font
+					(size 1.27 1.27)
+				)
+			)
+		)
 		(pin "1"
 		)
@@
 			)
 		)
+		(property "price" ".04"
+			(at 154.94 124.46 0)
+			(hide yes)
+			(show_name no)
+			(do_not_autoplace no)
+			(effects
+				(font
+					(size 1.27 1.27)
+				)
+			)
+		)
 		(pin "1"
 		)
@@
 			(hide yes)
 			(show_name no)
+			(do_not_autoplace no)
+			(effects
+				(font
+					(size 1.27 1.27)
+				)
+			)
+		)
+		(property "price" ".04"
+			(at 93.98 81.28 0)
+			(hide yes)
+			(show_name no)

Commit message: june_26
Parts:
- RL2: value 100 -> 50; symbol Resistors:0402_R100 -> Resistors:0402_R050; DN P100DECT-ND -> TNP49.9DACT-ND; MFR Panasonic Electronic Components -> Vishay Dale; MPN ERA-2AED101X -> TNPW040249R9BEED; price .04 -> .30
- W10, W11, W12, W7, W8, W9: value (none) -> splitter; DNP (none) -> DNP; now not fitted
Other:
- moved on the sheet: R10, R11, R12, R8, R9, RL2
