File: Microwave_Beamer.kicad_sch (KiCad schematic)
At the start: 10 parts, among them IC1 MAX2870ETJ+, Y1 ECS-3225MVQ-1000-CN-TR

Commit message: skdja7rkweg
Parts:
- added C135, C137, C138: 1uF, Capacitor_SMD:C_0603_1608Metric, symbol Capacitors:0603_uF001_50V
- added C280: 1nF, Capacitor_SMD:C_0402_1005Metric, symbol Capacitors:0402_nF1_50V
- added C281, C282, C322: 100nF, Capacitor_SMD:C_0603_1608Metric, symbol Capacitors:0603_nf100
- added C323, C324, C325, C326, C327, C328: 100nF, Capacitor_SMD:C_0402_1005Metric, symbol Capacitors:0402_nF100_50V
- added R43: 33, Resistor_SMD:R_0402_1005Metric, symbol Resistors:0402_R033
- added R44: 250, Resistor_SMD:R_0603_1608Metric, symbol Resistors:R
- added R45: 100, Resistor_SMD:R_0402_1005Metric, symbol Resistors:0402_R100
- added R48, R52, R53, R54, R55: 10K, Resistor_SMD:R_0603_1608Metric, symbol Resistors:0603_R_10K
Connections:
- net +3.3V: now also IC1.4 (CE), C322.1, C323.2, C324.2, C325.2, C326.2, C327.2, C328.2, R53.1
- net GND: now also Y1.1 (~{EN}), C135.1, C137.1, C138.1, C280.2, C282.2, C322.2, C323.1, C324.1, C325.1, C326.1, C327.1, C328.1, R45.2, R48.1, R52.1, R55.1
- net at IC1.19 (NOISE_FILT): now also C137.2
- net at IC1.20 (TUNE): now also C280.1, R44.2
- net at IC1.22 (RSET): now also R48.2, R52.2
- net at IC1.23 (BIAS_FILT): now also C135.2
- net at IC1.24 (REG): now also C138.2
- net at IC1.25 (LD): now also R54.2
- net at IC1.26 (RFOUT_EN): now also R53.2
- net at IC1.5 (SW): now also R43.2, R45.1
- net at IC1.7 (CP_OUT): now also C281.1, C282.1, R44.1
- new net: C281.2, R43.1
- new net: R54.1, R55.2
- no-connect marks 0 -> 2
Other:
- removed sheet DCDC
- added sheet POWER (power.kicad_sch)
- added sheet pico_interface (pico.kicad_sch)
- sheet POWER AMP6 ports: added VCC, power detect; removed none
- moved on the sheet: C1, RR3, Y1

Commit message: moving along
Parts:
- removed C281, C282: 100nF, Capacitor_SMD:C_0603_1608Metric, symbol Capacitors:0603_nf100
- removed R55: 10K, Resistor_SMD:R_0603_1608Metric, symbol Resistors:0603_R_10K
- added C329, C330: 100nF, Capacitor_SMD:C_0402_1005Metric, symbol Capacitors:0402_nF100_50V
- added D1, D2, D3, D4, D5, D6: LTST-C230KGKT, LED_SMD:LED_1206_3216Metric, symbol LED:IR26-21C_L110_TR8
- added R56, R57, R58, R59: 250, Resistor_SMD:R_0603_1608Metric, symbol Resistors:R
- added R60, R61: 100, Resistor_SMD:R_0402_1005Metric, symbol Resistors:0402_R100
- added U51, U53, U57: SN74LVC1G14DCKR, Logic:SOT65P210X110-5N, symbol Logic:SN74LVC1G14DCKR
- added U54: 74HC138D, Logic:SOT109-1_NXP, symbol Logic:74HC138D
- added U56: PI_PICO, Logic:PI_PICO_SMD, symbol Logic:PI_PICO
- R54: now fitted
- RR1, RR2, RR3, RR4, RR5, RR6: cost (none) -> .30
Connections:
- net 3V3 is gone; now on net +3.3V: RR1.1, RR2.1
- net +3.3V: now also R54.1, U51.5 (VCC), U53.5 (VCC); no longer IC1.4 (CE)
- net +5V: now also D6.2 (A), U57.5 (VCC)
- net GND: now also C330.1, U51.3 (GND), U53.3 (GND), U54.3 (A2), U54.4 (E*1), U54.5 (E*2), U54.8 (GND), U57.3 (GND)
- net PHASE_CTRL_1: now also U51.2 (A), U54.2 (A1), U56.16 (GP12)
- net PHASE_CTRL_2: now also U53.2 (A), U54.1 (A0), U56.15 (GP11)
- net ~{PHASE_CTRL_1}: now also U51.4 (Y)
- net ~{PHASE_CTRL_2}: now also U53.4 (Y)
- net at IC1.7 (CP_OUT), R44.1: now also C329.1, C330.2
- net at R43.1: now also C329.2
- net CLK: now reaches IC1.1 (CLK)
- net CLK: now also U56.4 (GP2)
- net MOSI: now reaches IC1.2 (DATA)
- net MOSI: now also U56.5 (GP3)
- net at IC1.25 (LD): no longer R54.2
- net RF_EN: now reaches IC1.26 (RFOUT_EN), R53.2
- net RF_EN: now also U56.10 (GP7)
- net LE: now reaches IC1.3 (LE)
- net LE: now also U56.7 (GP5)
- net MISO/SDO: now reaches IC1.30 (MUX_OUT)
- net MISO/SDO: now also U56.6 (GP4)
- new net: D5.1 (K), R60.1, R61.1
- new net: D5.2 (A), D6.1 (K)
- new net: D3.1 (K), R58.1
- new net: D1.1 (K), R56.1
- new net: D2.1 (K), R57.1
- new net: R60.2, R61.2, U57.4 (Y)
- new net: D4.1 (K), R59.1
- new net 5V_LP: D1.2 (A), D2.2 (A), D3.2 (A), D4.2 (A), U54.16 (VCC), U54.6 (E3), U56.39 (VSYS)
- new net AMP_enable: U57.2 (A)
- new net CHIP_EN: IC1.4 (CE), R54.2, U56.9 (GP6)
- new net Stage_1_power: U56.31 (GP26)
- new net Stage_2_power: U56.32 (GP27)
- new net led_n20: R56.2, U54.15 (Y*0)
- new net led_n45: R59.2, U54.12 (Y*3)
- new net led_p30: R58.2, U54.13 (Y*2)
- new net led_zero: R57.2, U54.14 (Y*1)
- no-connect marks 2 -> 7
Other:
- removed sheet pico_interface
- sheet POWER ports: added 3V3, AMP_enable; removed none
- moved on the sheet: R53

Commit message: 6 layers now
Parts:
- R45, R60, R61: price (none) -> .04
Changed lines of the file:
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@@
 			)
 		)
+		(property "price" ".04"
+			(at 144.78 96.52 0)
+			(hide yes)
+			(show_name no)
+			(do_not_autoplace no)
+			(effects
+				(font
+					(size 1.27 1.27)
+				)
+			)
+		)
 		(pin "2"
 		)
@@
 			)
 		)
+		(property "price" ".04"
+			(at 241.3 148.59 0)
+			(hide yes)
+			(show_name no)
+			(do_not_autoplace no)
+			(effects
+				(font
+					(size 1.27 1.27)
+				)
+			)
+		)
 		(pin "2"
 		)
@@
 			(hide yes)
 			(show_name no)
+			(do_not_autoplace no)
+			(effects
+				(font
+					(size 1.27 1.27)
+				)
+			)
+		)
+		(property "price" ".04"
+			(at 245.11 148.59 0)
+			(hide yes)
+			(show_name no)

Commit message: completed length matching
Parts:
- added C139, C176: 2.2pF, Capacitor_SMD:C_0402_1005Metric, symbol Capacitors:0402_pF2.2_50V
- C323, C324, C325, C326, C327, C328, C329, C330: cost .02 -> (none); price .388 -> .02
- R61: now not fitted
Connections:
- net POWER AMP6/RF_IN: now also C176.2; no longer RR6.2
- net POWER AMP6/RF_OUT: now also C139.1
- new net: C176.1, RR6.2
- new net STEM/IN: C139.2
Other:
- moved on the sheet: D1, D2, D3, D4, D5, D6, R60, RR4, RR5, RR6, U56, U57

Commit message: june_26
Parts:
- removed C322: 100nF, Capacitor_SMD:C_0603_1608Metric, symbol Capacitors:0603_nf100
- removed R44: 250, Resistor_SMD:R_0603_1608Metric, symbol Resistors:R
- added C177, C181, C182, C183: 2.2pF, Capacitor_SMD:C_0402_1005Metric_Pad0.74x0.62mm_HandSolder, symbol Capacitors:0402_pF002.2_50V
- added C322: 100nF, Capacitor_SMD:C_0402_1005Metric, symbol Capacitors:0402_nF100_50V
- added D7: 30V 1.1A, Pulsemedica_Diodes:CR_03-GS08_VIS, symbol Pulsemedica_Diodes:SL03-GS08
- added H1, H2, H3, H4, H5, H6, H7: Hole, L_mechanical:PTH_5mm, symbol L_Mechanical:Hole
- added J1, J2: SMA-J-P-H-ST-EM1, L_Connectors:SAMTEC_SMA-J-P-H-ST-EM1, symbol L_Connectors:SMA-J-P-H-ST-EM1
- added J3, J4, J5, J6, J7: 4pos_TH, L_Connectors:4POS-2_54-generic, symbol L_Connectors:4pos_TH
- added J8: PJ-002A, Pulsemedica_Connectors:CUI_PJ-002A, symbol Pulsemedica_Connectors:PJ-002A
- added R72: 10K, Resistor_SMD:R_0603_1608Metric, symbol Resistors:0603_R_10K
- added R74, R75, R76: 100, Resistor_SMD:R_0402_1005Metric, symbol Resistors:0402_R100
- added SW1, SW2: PTS526SM15SMTR2 LFS, L_mechanical:SON4_PTS526 SM15 SMTR2 LFS_CNK-M, symbol L_Mechanical:PTS526_SM15_SMTR2_LFS
- C1, C176, C2: symbol Capacitors:0402_pF2.2_50V -> Capacitors:0402_pF002.2_50V; price (none) -> .08
- C139: footprint Capacitor_SMD:C_0402_1005Metric -> Capacitor_SMD:C_0402_1005Metric_Pad0.74x0.62mm_HandSolder; symbol Capacitors:0402_pF2.2_50V -> Capacitors:0402_pF002.2_50V; price (none) -> .08
- C280: price (none) -> .07
- D1, D2, D3, D4: price (none) -> .19
- D5, D6: DN 160-1456-1-ND -> 160-1457-1-ND; MPN LTST-C230KGKT -> LTST-C230KRKT; price (none) -> .19; now not fitted
- IC1: price (none) -> 31.51
- R43: cost .30 -> (none); price (none) -> .30
- R48, R52, R53, R54: DN (none) -> P10KDBCT-ND; MFR (none) -> Panasonic Industry; MPN (none) -> ERA-3AEB103V; price (none) -> .1
- R56, R57, R58, R59: value 250 -> 1k; symbol Resistors:R -> Resistors:0603_R_01K; DN (none) -> P1.0KDBCT-ND; MFR (none) -> Panasonic Industry; MPN (none) -> ERA-3AEB102V; price (none) -> x
- R62: renamed from RR3; cost .30 -> (none); price (none) -> .30
- R63: renamed from RR1; cost .30 -> (none); price (none) -> .30
- R64: renamed from RR2; cost .30 -> (none); price (none) -> .30
- R65: renamed from RR4; cost .30 -> (none); price (none) -> .30
- R66: renamed from RR5; cost .30 -> (none); price (none) -> .30
- R67: renamed from RR6; cost .30 -> (none); price (none) -> .30
- Y1: price (none) -> 2.2
Connections:
- net +3.3V: now also C322.2, J3.3, J6.4, J7.4
- net +5V: now also H3.1, J4.2
- net 5V_LP: now also D7.A, J3.4; no longer U56.39 (VSYS)
- net CHIP_EN: now also J6.2
- net CLK: now also J5.1
- net GND: now also U56.13 (GND__2), U56.18 (GND__3), U56.23 (GND__4), U56.28 (GND__5), U56.3 (GND), U56.33 (AGND), U56.38 (GND__6), U56.8 (GND__1), U56.D2 (GND__7), C177.1, C181.1, C182.1, C183.2, C322.1, H2.1, H4.1, H5.1, H6.1, H7.1, J1.2_1, J1.2_2, J1.3_1, J1.3_2, J2.2_1, J2.2_2, J2.3_1, J2.3_2, J3.1, J4.1, J4.3, J6.1, J7.1, J8.2, SW1.3, SW1.4, SW2.3, SW2.4
- net LE: now also J5.4
- net MISO/SDO: now also J5.3
- net MOSI: now also J5.2
- net PHASE_CTRL_1: now also J7.3
- net PHASE_CTRL_2: now also J7.2
- net RF_EN: now also J6.3, R72.1
- net at C329.1, C330.2, IC1.7 (CP_OUT): now also R74.1
- net at C280.1, IC1.20 (TUNE): now also R76.2
- net BTN_1: now reaches U56.1 (GP0)
- net BTN_1: now also SW1.1, SW1.2
- net DCDC EN: now reaches U56.11 (GP8)
- net BTN_2: now reaches U56.2 (GP1)
- net BTN_2: now also SW2.1, SW2.2
- net AMP_enable: no longer names the net of U57.2 (A)
- net AMP_enable: now also R72.2
- new net: C183.1, J2.1
- new net: R74.2, R75.1
- new net: R75.2, R76.1
- new net: D7.K, U56.39 (VSYS)
- new net +12V: H1.1, J4.4, J8.1
- new net 2.85VREF: J3.2
- new net RF_IO: C177.2, J1.1
- new net ext_to_amp: C181.2, C182.2
- no-connect marks 7 -> 10
Other:
- sheet POWER ports: added 5V; removed none
- note added: "2V @ 10-20mA"
- note added: "2V @ 5-20mA"
- note added: "transform to 1Kohm"
- note removed: "look into dedicated attenuators"
- moved on the sheet: R65, R67
