File: Microwave_Beamer.kicad_sch (KiCad schematic)
At the start: 74 parts, among them IC1 MAX2870ETJ+, J1 SMA-J-P-H-ST-EM1, J2 SMA-J-P-H-ST-EM1, J3 4pos_TH, J4 4pos_TH, J5 4pos_TH, J6 4pos_TH, J7 4pos_TH, J8 PJ-002A, SW1 PTS526SM15SMTR2 LFS, SW2 PTS526SM15SMTR2 LFS, U51 SN74LVC1G14DCKR, U53 SN74LVC1G14DCKR, U54 74HC138D, U56 PI_PICO, U57 SN74LVC1G14DCKR, Y1 ECS-3225MVQ-1000-CN-TR

Commit message: created fab files, needs some cleanup
Parts:
- added C142: 2.2pF, Capacitor_SMD:C_0402_1005Metric_Pad0.74x0.62mm_HandSolder, symbol Capacitors:0402_pF002.2_50V
- added C331: 100nF, Capacitor_SMD:C_0402_1005Metric, symbol Capacitors:0402_nF100_50V
- added R77, R78: 50, Resistor_SMD:R_0402_1005Metric_Pad0.72x0.64mm_HandSolder, symbol Resistors:0402_R050
- added U58: LMH2120UM/NOPB, RF_components:RF_DETECT, symbol RF_components:LMH2120UM_NOPB
- D7: now fitted
Connections:
- net +3.3V: now also C331.1, U58.A1 (VDD), U58.C2 (EN)
- net GND: now also C331.2, R77.2, R78.2, U58.B2 (GND), U58.C1 (GND)
- net coupled power: now reaches U56.34 (GP28)
- net coupled power: now also U58.A2 (OUT)
- new net: C142.1, R78.1
- new net: C142.2, U58.B1 (RF_IN)
- no-connect marks 10 -> 11
Other:
- note added: "coupled line"
- moved on the sheet: D1, D2, D3, D4, R56, R57, R58, R59, U54

Commit message: created version with standard stackup
Parts:
- removed U58: LMH2120UM/NOPB, RF_components:RF_DETECT, symbol RF_components:LMH2120UM_NOPB
- added C282: 1nF, Capacitor_SMD:C_0402_1005Metric, symbol Capacitors:0402_nF1_50V
- added R79, R80: 1k, Resistor_SMD:R_0603_1608Metric, symbol Resistors:0603_R_01K
- added U59: LTC5531ES6-TRMPBF, RF_components:SOT-6_S_LIT-M, symbol RF_components:LTC5531ES6-TRMPBF
- U54: MPN 74HC138D,653 -> MC74HC138ADR2G; price .37 -> .64
- renumbered IC1 to U58, Y1 to X1
Connections:
- net +3.3V: now also C282.1, R80.2, U59.3 (*SHDN), U59.6 (VCC)
- net GND: now also C282.2, R79.2, U59.2 (GND)
- net coupled power: now also U59.5 (VOUT)
- net at C142.2: now also U59.1 (RFIN)
- new net: R79.1, R80.1, U59.4 (VOS)
Other:
- moved on the sheet: C331, R77

Commit message: updated bom
Parts:
- U54: DN 1727-2781-1-ND -> MC74HC138ADR2GOSCT-ND
Other:
- note added: "substitute: 5004L-R"
Changed lines of the file:
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@@
 		)
 	)
+	(text "substitute: 5004L-R"
+		(exclude_from_sim no)
+		(at 83.82 186.69 0)
+		(effects
+			(font
+				(size 1.27 1.27)
+			)
+		)
+	)
 	(junction
 		(at 66.04 43.18)
@@
 			)
 		)
-		(property "Description" "Decoder/Demultiplexer 1 x 3:8 16-SO"
+		(property "Description" "Decoder/Demultiplexer 1 x 3:8 16-SO substitute: MC74HC138ADR2G"
 			(at 33.02 165.1 0)
 			(hide yes)
@@
 			)
 		)
-		(property "DN" "1727-2781-1-ND"
+		(property "DN" "MC74HC138ADR2GOSCT-ND"
 			(at 33.02 162.56 0)
 			(hide yes)
