File: POWER_AMP2.kicad_sch (KiCad schematic)
At the start: 9 parts, among them U14 SE5023L-R

Commit message: skdja7rkweg
Parts:
- removed C12, C13: 1nF, Capacitor_SMD:C_0402_1005Metric, symbol Capacitors:0402_nF1_50V
- removed C14, C15: 100pF, Capacitor_SMD:C_0402_1005Metric, symbol Capacitors:0402_pF_100_50V
- removed C16, C262: 100pFX, Capacitor_SMD:C_0402_1005Metric, symbol Capacitors:0402_pF_100_50V
- added C12: 100nF, Capacitor_SMD:C_0603_1608Metric, symbol Capacitors:0603_nf100
- added C304: 10nF, Capacitor_SMD:C_0402_1005Metric, symbol Capacitors:0402_nF010_50V
- added C53: 1uF, Capacitor_SMD:C_0603_1608Metric, symbol Capacitors:0603_uF001_50V
Connections:
- net GND: now also C12.2, C304.2, C53.2
- net +5V renamed VCC
- net VCC: now also C12.1, C304.1, C53.1

Commit message: completed length matching
Parts:
- C12: footprint Capacitor_SMD:C_0603_1608Metric -> Capacitor_SMD:C_0402_1005Metric; symbol Capacitors:0603_nf100 -> Capacitors:0402_nF100_50V; DN 490-5798-1-ND -> 490-14514-1-ND; MPN GCJ188R71H104KA12D -> GCM155R71H104KE02J; price .10 -> .02
- C304: value 10nF -> 100nF; symbol Capacitors:0402_nF010_50V -> Capacitors:0402_nF100_50V; DN 490-4762-1-ND -> 490-14514-1-ND; MPN GCM155R71H103KA55D -> GCM155R71H104KE02J; price .388 -> .02
Other:
- moved on the sheet: C12
Changed lines of the file:
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@@
+	)
+	(junction
+		(at 96.52 86.36)
+		(diameter 0)
+		(color 0 0 0 0)
 	)
 	(junction
@@
 	)
 	(junction
-		(at 96.52 93.98)
-		(diameter 0)
-		(color 0 0 0 0)
-	)
-	(junction
 		(at 58.42 114.3)
 		(diameter 0)
@@
 	)
 	(junction
+		(at 104.14 86.36)
+		(diameter 0)
+		(color 0 0 0 0)
+	)
+	(junction
 		(at 111.76 93.98)
 		(diameter 0)
@@
 	)
 	(junction
-		(at 96.52 86.36)
+		(at 50.8 86.36)
 		(diameter 0)
 		(color 0 0 0 0)
 	)
 	(junction
-		(at 101.6 86.36)
-		(diameter 0)
-		(color 0 0 0 0)
-	)
-	(junction
-		(at 50.8 86.36)
+		(at 104.14 93.98)
 		(diameter 0)
 		(color 0 0 0 0)
@@
 	)
 	(junction
-		(at 101.6 93.98)
+		(at 96.52 93.98)
 		(diameter 0)
 		(color 0 0 0 0)
@@
 	(wire
 		(pts
-			(xy 101.6 86.36) (xy 96.52 86.36)
+			(xy 96.52 86.36) (xy 104.14 86.36)
 		)
 		(stroke
@@
 	(wire
 		(pts
-			(xy 101.6 93.98) (xy 111.76 93.98)
-		)
-		(stroke
-			(width 0)
-			(type default)
-		)
-	)
-	(wire
-		(pts
 			(xy 86.36 86.36) (xy 86.36 88.9)
 		)
@@
 	(wire
 		(pts
-			(xy 96.52 93.98) (xy 101.6 93.98)
+			(xy 96.52 93.98) (xy 104.14 93.98)
 		)
 		(stroke
@@
 	(wire
 		(pts
+			(xy 104.14 93.98) (xy 111.76 93.98)
+		)
+		(stroke
+			(width 0)
+			(type default)
+		)
+	)
+	(wire
+		(pts
 			(xy 58.42 114.3) (xy 60.96 114.3)
 		)
@@
 	(wire
 		(pts
+			(xy 104.14 86.36) (xy 111.76 86.36)
+		)
+		(stroke
+			(width 0)
+			(type default)
+		)
+	)
+	(wire
+		(pts
 			(xy 71.12 114.3) (xy 73.66 114.3)
 		)
@@
 		(pts
 			(xy 86.36 93.98) (xy 86.36 96.52)
-		)
-		(stroke
-			(width 0)
-			(type default)
-		)
-	)
-	(wire
-		(pts
-			(xy 101.6 86.36) (xy 111.76 86.36)
 		)
 		(stroke
@@
 	)
 	(symbol
-		(lib_id "Capacitors:0402_nF010_50V")
+		(lib_id "Capacitors:0402_nF100_50V")
 		(at 96.52 86.36 0)
 		(unit 1)
@@
 			)
 		)
-		(property "Value" "10nF"
-			(at 93.98 83.82 0)
-			(show_name no)
-			(do_not_autoplace no)
-			(effects
-				(font
-					(size 1.27 1.27)
-				)
-				(justify left)
+		(property "Value" "100nF"
+			(at 99.06 83.82 0)
+			(show_name no)
+			(do_not_autoplace no)
+			(effects
+				(font
+					(size 1.27 1.27)
+				)
 			)
 		)
@@
 			)
 		)
-		(property "Description" "10000 pF ±10% 50V Ceramic Capacitor X7R 0402 (1005 Metric)"
+		(property "Description" "0.1 µF ±10% 50V Ceramic Capacitor X7R 0402 (1005 Metric)"
 			(at 91.44 78.74 0)
 			(hide yes)
@@
 			)
 		)
-		(property "MPN" "GCM155R71H103KA55D"
+		(property "MPN" "GCM155R71H104KE02J"
 			(at 96.52 86.36 0)
 			(hide yes)
@@
 			)
 		)
-		(property "DN" "490-4762-1-ND"
+		(property "DN" "490-14514-1-ND"
 			(at 96.52 86.36 0)
 			(hide yes)
@@
 			)
 		)
-		(property "price" ".388"
+		(property "price" ".02"
 			(at 96.52 86.36 0)
 			(hide yes)
@@
 	)
 	(symbol
-		(lib_id "Capacitors:0603_nf100")
-		(at 101.6 86.36 0)
+		(lib_id "Capacitors:0402_nF100_50V")
+		(at 104.14 86.36 0)
 		(unit 1)
 		(body_style 1)
@@
 		(dnp no)
 		(property "Reference" "C12"
-			(at 101.6 81.28 0)
+			(at 104.14 81.28 0)
 			(show_name no)
 			(do_not_autoplace no)
@@
 		)
 		(property "Value" "100nF"
-			(at 101.6 83.82 0)
-			(show_name no)
-			(do_not_autoplace no)
-			(effects
-				(font
-					(size 1.27 1.27)
-				)
-				(justify left)
-			)
-		)
-		(property "Footprint" "Capacitor_SMD:C_0603_1608Metric"
-			(at 99.822 86.36 90)
-			(hide yes)
-			(show_name no)
-			(do_not_autoplace no)
-			(effects
-				(font
-					(size 1.27 1.27)
-				)
-			)
-		)
-		(property "Datasheet" ""
-			(at 95.25 83.185 0)
-			(hide yes)
-			(show_name no)
-			(do_not_autoplace no)
-			(effects
-				(font
-					(size 1.27 1.27)
-				)
-			)
-		)
-		(property "Description" "0.1 µF ±10% 50V Ceramic Capacitor X7R 0603 (1608 Metric)"
-			(at 96.52 78.74 0)
-			(hide yes)
-			(show_name no)
-			(do_not_autoplace no)
-			(effects
-				(font
-					(size 1.27 1.27)
-				)
-			)
-		)
-		(property "MPN" "GCJ188R71H104KA12D"
-			(at 101.6 86.36 0)
-			(hide yes)
-			(show_name no)
-			(do_not_autoplace no)
-			(effects
-				(font
-					(size 1.27 1.27)
-				)
-			)
-		)
-		(property "DN" "490-5798-1-ND"
-			(at 101.6 86.36 0)
+			(at 106.68 83.82 0)
+			(show_name no)
+			(do_not_autoplace no)
+			(effects
+				(font
+					(size 1.27 1.27)
+				)
+			)
+		)
+		(property "Footprint" "Capacitor_SMD:C_0402_1005Metric"
+			(at 102.362 86.36 90)
+			(hide yes)
+			(show_name no)
+			(do_not_autoplace no)
+			(effects
+				(font
+					(size 1.27 1.27)
+				)
+			)
+		)
+		(property "Datasheet" "https://ds.murata.com/simsurfing/mlcc.html?lcid=en-us&jis=false&md5=ffdf2ea84f2d70fe82acfb70297713ec"
+			(at 97.79 83.185 0)
+			(hide yes)
+			(show_name no)
+			(do_not_autoplace no)
+			(effects
+				(font
+					(size 1.27 1.27)
+				)
+			)
+		)
+		(property "Description" "0.1 µF ±10% 50V Ceramic Capacitor X7R 0402 (1005 Metric)"
+			(at 99.06 78.74 0)
+			(hide yes)
+			(show_name no)
+			(do_not_autoplace no)
+			(effects
+				(font
+					(size 1.27 1.27)
+				)
+			)
+		)
+		(property "MPN" "GCM155R71H104KE02J"
+			(at 104.14 86.36 0)
+			(hide yes)
+			(show_name no)
+			(do_not_autoplace no)
+			(effects
+				(font
+					(size 1.27 1.27)
+				)
+			)
+		)
+		(property "DN" "490-14514-1-ND"
+			(at 104.14 86.36 0)
 			(hide yes)
 			(show_name no)
@@
 		)
 		(property "MFR" "Murata Electronics"
-			(at 101.6 86.36 0)
-			(hide yes)
-			(show_name no)
-			(do_not_autoplace no)
-			(effects
-				(font
-					(size 1.27 1.27)
-				)
-			)
-		)
-		(property "price" ".10"
-			(at 101.6 86.36 0)
-			(hide yes)
-			(show_name no)
+			(at 104.14 86.36 0)
+			(hide yes)
+			(show_name no)
+			(do_not_autoplace no)
+			(effects
+				(font
+					(size 1.27 1.27)
+				)
+			)
+		)
+		(property "price" ".02"
+			(at 104.14 86.36 0)
+			(hide yes)
+			(show_name no)

Commit message: june_26
Parts:
- C10, C11: price (none) -> .07
- C304: cost .02 -> (none)
- U14: price (none) -> 6.3
Changed lines of the file:
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@@
 	(paper "A4")
+	(junction
+		(at 73.66 114.3)
+		(diameter 0)
+		(color 0 0 0 0)
+	)
 	(junction
 		(at 86.36 93.98)
@@
 	)
 	(junction
+		(at 66.04 114.3)
+		(diameter 0)
+		(color 0 0 0 0)
+	)
+	(junction
 		(at 96.52 86.36)
 		(diameter 0)
@@
 	)
 	(junction
-		(at 86.36 88.9)
+		(at 86.36 86.36)
 		(diameter 0)
 		(color 0 0 0 0)
 	)
 	(junction
-		(at 66.04 114.3)
+		(at 63.5 114.3)
+		(diameter 0)
+		(color 0 0 0 0)
+	)
+	(junction
+		(at 86.36 91.44)
 		(diameter 0)
 		(color 0 0 0 0)
@@
 	)
 	(junction
+		(at 104.14 86.36)
+		(diameter 0)
+		(color 0 0 0 0)
+	)
+	(junction
 		(at 71.12 114.3)
 		(diameter 0)
@@
 	)
 	(junction
-		(at 63.5 114.3)
+		(at 86.36 88.9)
+		(diameter 0)
+		(color 0 0 0 0)
+	)
+	(junction
+		(at 111.76 93.98)
 		(diameter 0)
 		(color 0 0 0 0)
@@
 	)
 	(junction
+		(at 104.14 93.98)
+		(diameter 0)
+		(color 0 0 0 0)
+	)
+	(junction
+		(at 96.52 93.98)
+		(diameter 0)
+		(color 0 0 0 0)
+	)
+	(junction
 		(at 68.58 114.3)
 		(diameter 0)
@@
 	)
 	(junction
-		(at 104.14 86.36)
-		(diameter 0)
-		(color 0 0 0 0)
-	)
-	(junction
-		(at 111.76 93.98)
-		(diameter 0)
-		(color 0 0 0 0)
-	)
-	(junction
-		(at 73.66 114.3)
+		(at 76.2 114.3)
 		(diameter 0)
 		(color 0 0 0 0)
@@
 		(color 0 0 0 0)
 	)
-	(junction
-		(at 104.14 93.98)
-		(diameter 0)
-		(color 0 0 0 0)
-	)
-	(junction
-		(at 76.2 114.3)
-		(diameter 0)
-		(color 0 0 0 0)
-	)
-	(junction
-		(at 86.36 91.44)
-		(diameter 0)
-		(color 0 0 0 0)
-	)
-	(junction
-		(at 96.52 93.98)
-		(diameter 0)
-		(color 0 0 0 0)
-	)
-	(junction
-		(at 86.36 86.36)
-		(diameter 0)
-		(color 0 0 0 0)
-	)
 	(no_connect
 		(at 50.8 91.44)
 	)
 	(no_connect
+		(at 50.8 93.98)
+	)
+	(no_connect
 		(at 50.8 96.52)
-	)
-	(no_connect
-		(at 50.8 93.98)
 	)
 	(wire
@@
 	(wire
 		(pts
-			(xy 45.72 86.36) (xy 50.8 86.36)
+			(xy 86.36 93.98) (xy 86.36 96.52)
 		)
 		(stroke
@@
 	(wire
 		(pts
-			(xy 86.36 86.36) (xy 86.36 88.9)
+			(xy 60.96 114.3) (xy 63.5 114.3)
 		)
 		(stroke
@@
 	(wire
 		(pts
-			(xy 96.52 86.36) (xy 91.44 86.36)
+			(xy 76.2 114.3) (xy 78.74 114.3)
 		)
 		(stroke
@@
 	(wire
 		(pts
-			(xy 73.66 114.3) (xy 76.2 114.3)
+			(xy 96.52 86.36) (xy 91.44 86.36)
 		)
 		(stroke
@@
 	(wire
 		(pts
-			(xy 96.52 93.98) (xy 104.14 93.98)
+			(xy 45.72 86.36) (xy 50.8 86.36)
 		)
 		(stroke
@@
 	(wire
 		(pts
-			(xy 66.04 114.3) (xy 68.58 114.3)
+			(xy 96.52 93.98) (xy 104.14 93.98)
 		)
 		(stroke
@@
 	(wire
 		(pts
-			(xy 86.36 86.36) (xy 91.44 86.36)
+			(xy 73.66 114.3) (xy 76.2 114.3)
 		)
 		(stroke
@@
 	(wire
 		(pts
-			(xy 104.14 93.98) (xy 111.76 93.98)
+			(xy 86.36 86.36) (xy 91.44 86.36)
 		)
 		(stroke
@@
 	(wire
 		(pts
-			(xy 58.42 114.3) (xy 60.96 114.3)
+			(xy 104.14 93.98) (xy 111.76 93.98)
 		)
 		(stroke
@@
 	(wire
 		(pts
-			(xy 86.36 91.44) (xy 86.36 93.98)
+			(xy 68.58 114.3) (xy 71.12 114.3)
 		)
 		(stroke
@@
 	(wire
 		(pts
-			(xy 43.18 101.6) (xy 50.8 101.6)
+			(xy 86.36 91.44) (xy 86.36 93.98)
 		)
 		(stroke
@@
 	(wire
 		(pts
-			(xy 76.2 114.3) (xy 78.74 114.3)
+			(xy 58.42 114.3) (xy 60.96 114.3)
 		)
 		(stroke
@@
 	(wire
 		(pts
-			(xy 71.12 114.3) (xy 73.66 114.3)
+			(xy 50.8 86.36) (xy 50.8 88.9)
 		)
 		(stroke
@@
 	(wire
 		(pts
-			(xy 50.8 86.36) (xy 50.8 88.9)
+			(xy 71.12 114.3) (xy 73.66 114.3)
 		)
 		(stroke
@@
 	(wire
 		(pts
-			(xy 68.58 114.3) (xy 71.12 114.3)
+			(xy 90.17 101.6) (xy 86.36 101.6)
 		)
 		(stroke
@@
 	(wire
 		(pts
-			(xy 86.36 93.98) (xy 86.36 96.52)
+			(xy 86.36 86.36) (xy 86.36 88.9)
 		)
 		(stroke
@@
 	(wire
 		(pts
-			(xy 60.96 114.3) (xy 63.5 114.3)
+			(xy 66.04 114.3) (xy 68.58 114.3)
+		)
+		(stroke
+			(width 0)
+			(type default)
+		)
+	)
+	(wire
+		(pts
+			(xy 43.18 101.6) (xy 50.8 101.6)
 		)
 		(stroke
@@
 	(hierarchical_label "RF_OUT"
 		(shape input)
-		(at 86.36 101.6 0)
+		(at 90.17 101.6 0)
 		(effects
 			(font
@@
 			)
 			(justify left)
+		)
+	)
+	(netclass_flag ""
+		(length 2.54)
+		(shape round)
+		(at 45.72 101.6 180)
+		(fields_autoplaced yes)
+		(effects
+			(font
+				(size 1.27 1.27)
+			)
+			(justify right bottom)
+		)
+		(property "Net Class" "50 ohm"
+			(at 46.4185 104.14 0)
+			(show_name no)
+			(do_not_autoplace no)
+			(effects
+				(font
+					(size 1.27 1.27)
+				)
+				(justify left)
+			)
+		)
+		(property "Component Class" ""
+			(at 44.45 30.48 0)
+			(show_name no)
+			(do_not_autoplace no)
+			(effects
+				(font
+					(size 1.27 1.27)
+					(italic yes)
+				)
+			)
 		)
 	)
@@
 			)
 		)
+		(property "price" "6.3"
+			(at 50.8 83.82 0)
+			(hide yes)
+			(show_name no)
+			(do_not_autoplace no)
+			(effects
+				(font
+					(size 1.27 1.27)
+				)
+			)
+		)
 		(pin "13"
 		)
@@
 			)
 		)
-		(property "cost" ".02"
+		(property "cost" ""
 			(at 96.52 86.36 0)
 			(hide yes)
@@
 		(property "DN" "490-GCM1555C1H102GA16JCT-ND"
 			(at 92.71 74.93 0)
+			(hide yes)
+			(show_name no)
+			(do_not_autoplace no)
+			(effects
+				(font
+					(size 1.27 1.27)
+				)
+			)
+		)
+		(property "price" ".07"
+			(at 91.44 86.36 0)
 			(hide yes)
 			(show_name no)
@@
 			(hide yes)
 			(show_name no)
+			(do_not_autoplace no)
+			(effects
+				(font
+					(size 1.27 1.27)
+				)
+			)
+		)
+		(property "price" ".07"
+			(at 45.72 86.36 0)
+			(hide yes)
+			(show_name no)
