File: POWER_AMP2.kicad_sch (KiCad schematic)
At the start: 6 parts, among them U14 SE5023L-R

Commit message: created fab files, needs some cleanup
Parts:
- C11: value 1nF -> 100nF; symbol Capacitors:0402_nF1_50V -> Capacitors:0402_nF100_50V; DN 490-GCM1555C1H102GA16JCT-ND -> 490-14514-1-ND; MFR (none) -> Murata Electronics; MPN GCM1555C1H102GA16J -> GCM155R71H104KE02J; price .07 -> .02
- C53: now not fitted
Changed lines of the file:
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@@
 		(on_board yes)
 		(in_pos_files yes)
-		(dnp no)
+		(dnp yes)
 		(property "Reference" "C53"
 			(at 109.22 81.28 0)
@@
 	)
 	(symbol
-		(lib_id "Capacitors:0402_nF1_50V")
+		(lib_id "Capacitors:0402_nF100_50V")
 		(at 91.44 86.36 0)
 		(unit 1)
@@
 			)
 		)
-		(property "Value" "1nF"
+		(property "Value" "100nF"
 			(at 91.44 83.82 0)
 			(show_name no)
@@
 		)
 		(property "Footprint" "Capacitor_SMD:C_0402_1005Metric"
-			(at 90.17 76.2 0)
-			(hide yes)
-			(show_name no)
-			(do_not_autoplace no)
-			(effects
-				(font
-					(size 1.27 1.27)
-				)
-			)
-		)
-		(property "Datasheet" ""
+			(at 89.662 86.36 90)
+			(hide yes)
+			(show_name no)
+			(do_not_autoplace no)
+			(effects
+				(font
+					(size 1.27 1.27)
+				)
+			)
+		)
+		(property "Datasheet" "https://ds.murata.com/simsurfing/mlcc.html?lcid=en-us&jis=false&md5=ffdf2ea84f2d70fe82acfb70297713ec"
 			(at 85.09 83.185 0)
 			(hide yes)
@@
 			)
 		)
-		(property "Description" "1000 pF ±2% 50V Ceramic Capacitor C0G, NP0 0402 (1005 Metric)"
+		(property "Description" "0.1 µF ±10% 50V Ceramic Capacitor X7R 0402 (1005 Metric)"
 			(at 86.36 78.74 0)
 			(hide yes)
@@
 			)
 		)
-		(property "MPN" "GCM1555C1H102GA16J"
-			(at 92.71 74.93 0)
-			(hide yes)
-			(show_name no)
-			(do_not_autoplace no)
-			(effects
-				(font
-					(size 1.27 1.27)
-				)
-			)
-		)
-		(property "DN" "490-GCM1555C1H102GA16JCT-ND"
-			(at 92.71 74.93 0)
-			(hide yes)
-			(show_name no)
-			(do_not_autoplace no)
-			(effects
-				(font
-					(size 1.27 1.27)
-				)
-			)
-		)
-		(property "price" ".07"
+		(property "MPN" "GCM155R71H104KE02J"
 			(at 91.44 86.36 0)
 			(hide yes)
+			(show_name no)
+			(do_not_autoplace no)
+			(effects
+				(font
+					(size 1.27 1.27)
+				)
+			)
+		)
+		(property "DN" "490-14514-1-ND"
+			(at 91.44 86.36 0)
+			(hide yes)
+			(show_name no)
+			(do_not_autoplace no)
+			(effects
+				(font
+					(size 1.27 1.27)
+				)
+			)
+		)
+		(property "price" ".02"
+			(at 91.44 86.36 0)
+			(hide yes)
+			(show_name no)
+			(do_not_autoplace no)
+			(effects
+				(font
+					(size 1.27 1.27)
+				)
+			)
+		)
+		(property "MFR" "Murata Electronics"
+			(at 91.44 86.36 0)
+			(hide yes)

Commit message: updated bom
Parts:
- U14: DN 863-SE5023L-RCT-ND -> 863-1376-1-ND; MPN SE5023L-R -> 5004L-R
Other:
- note added: "substitute: 5004L-R"
Changed lines of the file:
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@@
 	(generator_version "10.0")
 	(paper "A4")
+	(text "substitute: 5004L-R"
+		(exclude_from_sim no)
+		(at 95.25 111.76 0)
+		(effects
+			(font
+				(size 1.27 1.27)
+			)
+		)
+	)
 	(junction
 		(at 73.66 114.3)
@@
 			)
 		)
-		(property "Description" "8.15-1.85GHz power amp"
+		(property "Description" "8.15-1.85GHz power amp substitute: 5004L-R"
 			(at 71.374 47.498 0)
 			(hide yes)
@@
 			)
 		)
-		(property "MPN" "SE5023L-R"
+		(property "MPN" "5004L-R"
 			(at 64.008 51.562 0)
 			(hide yes)
@@
 			)
 		)
-		(property "DN" "863-SE5023L-RCT-ND"
+		(property "DN" "863-1376-1-ND"
 			(at 71.374 47.498 0)
 			(hide yes)
