File: Stage_A.kicad_sch (KiCad schematic)
At the start: 49 parts, among them U1 SKY13575-639LF, U10 SKY13575-639LF, U11 SKY13575-639LF, U12 SKY13575-639LF, U2 SKY13575-639LF, U3 SKY13575-639LF, U4 SKY13575-639LF, U5 SKY13575-639LF, U6 SKY13575-639LF, U7 SKY13575-639LF, U8 SKY13575-639LF, U9 SKY13575-639LF

Commit message: created fab files, needs some cleanup
Connections:
- no-connect marks 0 -> 1
Other:
- sheet FAN_B ports: added power_det; removed none
Changed lines of the file:
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@@
 		(color 0 0 0 0)
 	)
+	(no_connect
+		(at 254 33.02)
+	)
 	(wire
 		(pts
@@
 	(wire
 		(pts
+			(xy 254 33.02) (xy 256.54 33.02)
+		)
+		(stroke
+			(width 0)
+			(type default)
+		)
+	)
+	(wire
+		(pts
 			(xy 50.8 101.6) (xy 50.8 124.46)
 		)
@@
 	(wire
 		(pts
+			(xy 254 58.42) (xy 256.54 58.42)
+		)
+		(stroke
+			(width 0)
+			(type default)
+		)
+	)
+	(wire
+		(pts
 			(xy 81.28 68.58) (xy 76.2 68.58)
 		)
@@
 		)
 	)
+	(global_label "Stage_2_power"
+		(shape input)
+		(at 254 58.42 180)
+		(fields_autoplaced yes)
+		(effects
+			(font
+				(size 1.27 1.27)
+			)
+			(justify right)
+		)
+		(property "Intersheetrefs" "${INTERSHEET_REFS}"
+			(at 237.045 58.42 0)
+			(hide yes)
+			(show_name no)
+			(do_not_autoplace no)
+			(effects
+				(font
+					(size 1.27 1.27)
+				)
+				(justify right)
+			)
+		)
+	)
 	(global_label "PHASE_CTRL_2"
 		(shape input)
@@
 		)
 	)
-	(global_label "Stage_2_power"
-		(shape input)
-		(at 256.54 33.02 180)
-		(fields_autoplaced yes)
-		(effects
-			(font
-				(size 1.27 1.27)
-			)
-			(justify right)
-		)
-		(property "Intersheetrefs" "${INTERSHEET_REFS}"
-			(at 239.585 33.02 0)
-			(hide yes)
-			(show_name no)
-			(do_not_autoplace no)
-			(effects
-				(font
-					(size 1.27 1.27)
-				)
-				(justify right)
-			)
-		)
-	)
 	(global_label "PHASE_CTRL_1"
 		(shape input)
@@
 			(effects
 				(font
+					(size 1.27 1.27)
+				)
+				(justify left)
+			)
+		)
+		(pin "power_det" output
+			(at 256.54 58.42 180)
+			(effects
+				(font
