File: power.kicad_sch (KiCad schematic)
At the start: 42 parts, among them U50 LDL1117S33R, U52 MIC5219-2.85YM5-TR, U55 TPS548D26RXXR

Commit message: created fab files, needs some cleanup
Other:
- note added: "DCDC TPS548 5V 40A"
- note added: "DCDC module 5V 1A"
- note added: "LDO LIN REG"
- note added: "LIN REG"
Changed lines of the file:
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@@
+		)
+	)
+	(text "LIN REG"
+		(exclude_from_sim no)
+		(at 87.376 -6.858 0)
+		(effects
+			(font
+				(size 1.27 1.27)
+			)
 		)
 	)
@@
 		)
 	)
+	(text "DCDC\nmodule\n5V 1A "
+		(exclude_from_sim no)
+		(at 68.326 -5.588 0)
+		(effects
+			(font
+				(size 1.27 1.27)
+			)
+		)
+	)
 	(text "Cin: 1uF\nCout 4.7uF+"
 		(exclude_from_sim no)
@@
 		)
 	)
+	(text "LDO\nLIN REG"
+		(exclude_from_sim no)
+		(at 106.172 -5.842 0)
+		(effects
+			(font
+				(size 1.27 1.27)
+			)
+		)
+	)
 	(text "10 mA max on PG"
 		(exclude_from_sim no)
@@
 		)
 	)
+	(text "DCDC\nTPS548\n5V 40A"
+		(exclude_from_sim no)
+		(at 68.58 -18.415 0)
+		(effects
+			(font
+				(size 1.27 1.27)
+			)
+		)
+	)
 	(text "12V"
 		(exclude_from_sim no)
@@
 	(text_box "switches: 10uA x8 \n2.85 LDO: 360mA\nVCO: 150mA \nXO: 30mA\nP=1.7*.541=920mW\n"
 		(exclude_from_sim no)
-		(at 105.41 74.93 0)
+		(at 92.71 79.3132 0)
 		(size 24.13 12.1268)
 		(margins 0.9525 0.9525 0.9525 0.9525)
@@
 		)
 	)
+	(polyline
+		(pts
+			(xy 81.28 -20.32) (xy 82.55 -19.05)
+		)
+		(stroke
+			(width 0)
+			(type default)
+			(color 255 0 5 1)
+		)
+	)
+	(polyline
+		(pts
+			(xy 81.28 -17.78) (xy 82.55 -19.05)
+		)
+		(stroke
+			(width 0)
+			(type default)
+			(color 255 0 5 1)
+		)
+	)
 	(wire
 		(pts
@@
 		)
 	)
+	(polyline
+		(pts
+			(xy 81.28 -20.32) (xy 82.55 -19.05)
+		)
+		(stroke
+			(width 0)
+			(type default)
+			(color 255 0 5 1)
+		)
+	)
 	(wire
 		(pts
@@
 		)
 	)
+	(polyline
+		(pts
+			(xy 93.98 1.27) (xy 95.25 2.54)
+		)
+		(stroke
+			(width 0)
+			(type default)
+			(color 255 0 5 1)
+		)
+	)
+	(polyline
+		(pts
+			(xy 119.38 -5.08) (xy 120.65 -6.35)
+		)
+		(stroke
+			(width 0)
+			(type default)
+			(color 255 0 5 1)
+		)
+	)
 	(wire
 		(pts
@@
 		)
 	)
+	(polyline
+		(pts
+			(xy 95.25 2.54) (xy 96.52 1.27)
+		)
+		(stroke
+			(width 0)
+			(type default)
+			(color 255 0 5 1)
+		)
+	)
 	(wire
 		(pts
@@
 		)
 	)
+	(polyline
+		(pts
+			(xy 95.25 2.54) (xy 96.52 1.27)
+		)
+		(stroke
+			(width 0)
+			(type default)
+			(color 255 0 5 1)
+		)
+	)
 	(wire
 		(pts
@@
 		)
 	)
+	(polyline
+		(pts
+			(xy 119.38 -5.08) (xy 120.65 -6.35)
+		)
+		(stroke
+			(width 0)
+			(type default)
+			(color 255 0 5 1)
+		)
+	)
 	(wire
 		(pts
@@
 	(polyline
 		(pts
+			(xy 76.2 2.54) (xy 77.47 1.27)
+		)
+		(stroke
+			(width 0)
+			(type default)
+			(color 255 0 5 1)
+		)
+	)
+	(polyline
+		(pts
 			(xy 73.66 -6.35) (xy 82.55 -6.35)
 		)
@@
 		)
 	)
+	(polyline
+		(pts
+			(xy 119.38 -7.62) (xy 120.65 -6.35)
+		)
+		(stroke
+			(width 0)
+			(type default)
+			(color 255 0 5 1)
+		)
+	)
 	(wire
 		(pts
@@
 		)
 	)
+	(polyline
+		(pts
+			(xy 74.93 1.27) (xy 76.2 2.54)
+		)
+		(stroke
+			(width 0)
+			(type default)
+			(color 255 0 5 1)
+		)
+	)
 	(wire
 		(pts
@@
 		)
 	)
+	(polyline
+		(pts
+			(xy 81.28 -17.78) (xy 82.55 -19.05)
+		)
+		(stroke
+			(width 0)
+			(type default)
+			(color 255 0 5 1)
+		)
+	)
 	(wire
 		(pts
@@
 		)
 	)
+	(polyline
+		(pts
+			(xy 76.2 2.54) (xy 77.47 1.27)
+		)
+		(stroke
+			(width 0)
+			(type default)
+			(color 255 0 5 1)
+		)
+	)
 	(wire
 		(pts
@@
 		)
 	)
+	(polyline
+		(pts
+			(xy 93.98 1.27) (xy 95.25 2.54)
+		)
+		(stroke
+			(width 0)
+			(type default)
+			(color 255 0 5 1)
+		)
+	)
 	(wire
 		(pts
@@
 		)
 	)
+	(polyline
+		(pts
+			(xy 74.93 1.27) (xy 76.2 2.54)
+		)
+		(stroke
+			(width 0)
+			(type default)
+			(color 255 0 5 1)
+		)
+	)
 	(wire
 		(pts
@@
 		)
 		(stroke
+			(width 0)
+			(type default)
+			(color 255 0 5 1)
+		)
+	)
+	(polyline
+		(pts
+			(xy 119.38 -7.62) (xy 120.65 -6.35)
+		)
+		(stroke

Commit message: created version with standard stackup
Parts:
- U50: DN 497-17239-1-ND -> 4878-LDI1117-3.3HCT-ND; MPN LDL1117S33R -> LDL1117S33R (LDI1117-3.3H); price .45 -> .26
- renumbered PS1 to U60
Changed lines of the file:
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@@
 			)
 		)
-		(property "MPN" "LDL1117S33R"
+		(property "MPN" "LDL1117S33R (LDI1117-3.3H)"
 			(at 53.34 60.96 0)
 			(hide yes)
@@
 			)
 		)
-		(property "DN" "497-17239-1-ND"
+		(property "DN" "4878-LDI1117-3.3HCT-ND"
 			(at 55.88 60.96 0)
 			(hide yes)
@@
 			)
 		)
-		(property "price" ".45"
+		(property "price" ".26"
 			(at 53.34 60.96 0)
 			(hide yes)
@@
 		(dnp no)
 		(fields_autoplaced yes)
-		(property "Reference" "PS1"
+		(property "Reference" "U60"
 			(at 55.88 33.02 0)
 			(show_name no)
@@
 			(project "Microwave_Beamer"
 				(path "/3d000777-5a6c-48c2-9bdf-76c34ab20cc7/9ae7c201-9480-402d-a0c4-3941bcca95cf"
-					(reference "PS1")
+					(reference "U60")
 					(unit 1)
 				)

Commit message: updated bom
Parts:
- C126, C127, C128, C130, C132, C133, C186, C188, C189, C190, C191, C193: DN 490-12456-1-ND -> 490-GRT31CR6YA106KE01KCT-ND; MPN GRT31CR61H106KE01L -> GRT31CR6YA106KE01K; cap@V (none) -> 5V: 8.5u | 12V: 3.6u | 24V: 1.5u; price .388 -> .324
- CB13: symbol Capacitors:1206_uF10 -> Capacitors:1206_uF010; DN 490-12456-1-ND -> 490-GRT31CR6YA106KE01KCT-ND; MPN GRT31CR61H106KE01L -> GRT31CR6YA106KE01K; cap@V (none) -> 5V: 8.5u | 12V: 3.6u | 24V: 1.5u; price .388 -> .324
- R47: value 75k -> 56k; symbol Resistors:0603_R_75k -> Resistors:0603_R_56K; DN P75KDBCT-ND -> P56KDBCT-ND; MPN ERA-3AEB753V -> ERA-3AEB563V; price .1 -> .16
Other:
- note added: "OG: TPS548D26RXXR (40A) VFB = 0.6V"
- note added: "Subdtitute: TPS548C26RXXR VFB = 0.8V"
